File: KDT_Hierarchical/Section A - Title A.kicad_sch (KiCad schematic)
At the start: 0 parts

Commit message: removed old title
Other:
- title: MCU - Power -> Sheet Title A
Changed lines of the file:
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@@
   (paper "A4")
   (title_block
-    (title "MCU - Power")
+    (title "Sheet Title A")
     (date "Last Modified Date")
     (rev "${REVISION}")
