File: KDT_Hierarchical/Section B - TItle B.kicad_sch (KiCad schematic)
At the start: 0 parts

Commit message: removed old title
Other:
- title: MCU - I/Os -> Sheet Title B
Changed lines of the file:
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@@
   (paper "A3")
   (title_block
-    (title "MCU - I/Os")
+    (title "Sheet Title B")
     (date "Last Modified Date")
     (rev "${REVISION}")
