File: KDT_Hierarchical/KDT_Hierarchical.kicad_pcb (KiCad board)
At the start: 6 copper layers, 0 parts

Commit message: removed old title
Other:
- board text added: "??mm"
- board text added: "??mm (??oz)"
- board text added: "L1 (??)"
- board text added: "L2 (??)"
- board text added: "L3 (??"
- board text added: "L4 (??)"
- board text added: "L5 (??)"
- board text added: "L6 (??)"
- board text removed: "0.035mm (1oz)"
- board text removed: "0.07mm (2oz)"
- board text removed: "0.18mm"
- board text removed: "0.4mm"
- board text removed: "L1 (Sig, PWR)"
- board text removed: "L2 (GND)"
- board text removed: "L3 (Sig, PWR)"
- board text removed: "L4 (Sig, PWR)"
- board text removed: "L5 (GND)"
- board text removed: "L6 (Sig, PWR)"
Changed lines of the file:
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@@
     (effects (font (size 1 1) (thickness 0.2) bold) (justify left))
   )
-  (gr_text "L4 (Sig, PWR)" (at 51.5 86.5) (layer "User.4")
+  (gr_text "L4 (??)" (at 51.5 86.5) (layer "User.4")
     (effects (font (size 1 1) (thickness 0.2) bold) (justify left))
   )
@@
     (effects (font (size 1 1) (thickness 0.2) bold) (justify left))
   )
-  (gr_text "0.4mm" (at 65 90.75) (layer "User.4")
-    (effects (font (size 1 1) (thickness 0.125)) (justify left))
-  )
-  (gr_text "L3 (Sig, PWR)" (at 51.5 80) (layer "User.4")
+  (gr_text "??mm" (at 65 90.75) (layer "User.4")
+    (effects (font (size 1 1) (thickness 0.125)) (justify left))
+  )
+  (gr_text "L3 (??" (at 51.5 80) (layer "User.4")
     (effects (font (size 1 1) (thickness 0.2) bold) (justify left))
   )
@@
     (effects (font (size 1 1) (thickness 0.125)) (justify left))
   )
-  (gr_text "L2 (GND)" (at 51.5 71.5) (layer "User.4")
+  (gr_text "L2 (??)" (at 51.5 71.5) (layer "User.4")
     (effects (font (size 1 1) (thickness 0.2) bold) (justify left))
   )
@@
     (effects (font (size 1 1) (thickness 0.125)) (justify left))
   )
-  (gr_text "L6 (Sig, PWR)" (at 51.5 101.75) (layer "User.4")
+  (gr_text "L6 (??)" (at 51.5 101.75) (layer "User.4")
     (effects (font (size 1 1) (thickness 0.2) bold) (justify left))
   )
@@
     (effects (font (size 1 1) (thickness 0.2) bold) (justify left))
   )
-  (gr_text "0.035mm (1oz)" (at 65 86.5) (layer "User.4")
+  (gr_text "??mm (??oz)" (at 65 86.5) (layer "User.4")
     (effects (font (size 1 1) (thickness 0.2) bold) (justify left))
   )
@@
     (effects (font (size 1 1) (thickness 0.125)) (justify left))
   )
-  (gr_text "0.035mm (1oz)" (at 65 95) (layer "User.4")
-    (effects (font (size 1 1) (thickness 0.2) bold) (justify left))
-  )
-  (gr_text "0.18mm" (at 65 98.25) (layer "User.4")
+  (gr_text "??mm (??oz)" (at 65 95) (layer "User.4")
+    (effects (font (size 1 1) (thickness 0.2) bold) (justify left))
+  )
+  (gr_text "??mm" (at 65 98.25) (layer "User.4")
     (effects (font (size 1 1) (thickness 0.125)) (justify left))
   )
@@
     (effects (font (size 1 1) (thickness 0.125)) (justify left))
   )
-  (gr_text "0.18mm" (at 65 68.25) (layer "User.4")
-    (effects (font (size 1 1) (thickness 0.125)) (justify left))
-  )
-  (gr_text "0.18mm" (at 65 83.25) (layer "User.4")
+  (gr_text "??mm" (at 65 68.25) (layer "User.4")
+    (effects (font (size 1 1) (thickness 0.125)) (justify left))
+  )
+  (gr_text "??mm" (at 65 83.25) (layer "User.4")
     (effects (font (size 1 1) (thickness 0.125)) (justify left))
   )
@@
     (effects (font (size 1 1) (thickness 0.125)) (justify left))
   )
-  (gr_text "0.035mm (1oz)" (at 65 80) (layer "User.4")
+  (gr_text "??mm (??oz)" (at 65 80) (layer "User.4")
     (effects (font (size 1 1) (thickness 0.2) bold) (justify left))
   )
@@
     (effects (font (size 1 1) (thickness 0.125)) (justify left))
   )
-  (gr_text "0.07mm (2oz)" (at 65 64.75) (layer "User.4")
-    (effects (font (size 1 1) (thickness 0.2) bold) (justify left))
-  )
-  (gr_text "L1 (Sig, PWR)" (at 51.5 64.75) (layer "User.4")
+  (gr_text "??mm (??oz)" (at 65 64.75) (layer "User.4")
+    (effects (font (size 1 1) (thickness 0.2) bold) (justify left))
+  )
+  (gr_text "L1 (??)" (at 51.5 64.75) (layer "User.4")
     (effects (font (size 1 1) (thickness 0.2) bold) (justify left))
   )
@@
     (effects (font (size 1 1) (thickness 0.125)) (justify left))
   )
-  (gr_text "0.4mm" (at 65 75.75) (layer "User.4")
+  (gr_text "??mm" (at 65 75.75) (layer "User.4")
     (effects (font (size 1 1) (thickness 0.125)) (justify left))
   )
@@
     (effects (font (size 1 1) (thickness 0.15)) (justify left bottom))
   )
-  (gr_text "0.07mm (2oz)" (at 65 101.75) (layer "User.4")
-    (effects (font (size 1 1) (thickness 0.2) bold) (justify left))
-  )
-  (gr_text "L5 (GND)" (at 51.5 95) (layer "User.4")
+  (gr_text "??mm (??oz)" (at 65 101.75) (layer "User.4")
+    (effects (font (size 1 1) (thickness 0.2) bold) (justify left))
+  )
+  (gr_text "L5 (??)" (at 51.5 95) (layer "User.4")
     (effects (font (size 1 1) (thickness 0.2) bold) (justify left))
   )
@@
     (effects (font (size 1 1) (thickness 0.2) bold) (justify left))
   )
-  (gr_text "0.035mm (1oz)" (at 65 71.5) (layer "User.4")
-    (effects (font (size 1 1) (thickness 0.2) bold) (justify left))
-  )
+  (gr_text "??mm (??oz)" (at 65 71.5) (layer "User.4")
+    (effects (font (size 1 1) (thickness 0.2) bold) (justify left))
+  )

Commit message: Updated PCB
Other:
- board text added: "??? ??? ???"
- board text added: "??? ??? ??? ??? ??? (slot) ??? ??? ??? ??? ???"
- board text added: "???mm"
- board text added: "???mm (?oz)"
- board text added: "???mm ???mm ???mm ???mm ???mm ???mm ???mm ???mm ???mm ???mm"
- board text added: "ASSEMBLY NOTES (UNLESS OTHERWISE SPECIFIED) 1) DO NOT POPULATE PARTS ARE MARKED WITH A RED CROSS. 2) DO NOT POPULATE PARTS ARE NOT PRESENT IN THE BOM. 3) IF CONFLICTING INFORMATION IS FOUND BETWEEN THE ASSEMBLY FILE AND BOM, BOM SHOULD BE USED AS THE MAIN SOURCE."
- board text added: "Back Side"
- board text added: "Bottom Assembly (Scale 1:1)"
- board text added: "Bottom Fabrication (Scale 1:1)"
- board text added: "Bottom Test Points (Scale 1:1)"
- board text added: "Bottom View"
- board text added: "Components"
- board text added: "Count"
- board text added: "Drill Drawing (Top View) (Scale 1:1)"
- board text added: "FABRICATION NOTES (UNLESS OTHERWISE SPECIFIED) 1) OUTLINE DEFINED IN SEPARATE GERBER FILE WITH {dblquote}Edge_Cuts.GBR{dblquote} SUFFIX. DIMENSIONS OF CIRCUMSIZED RECTANGLE SHOWN ON THIS DWG FOR REF ONLY. 2) SEE SEPARATE DRILL FILES WITH {dblquote}.DRL{dblquote} SUFFIX FOR HOLE LOCATIONS. SELECTED HOLE LOCATIONS SHOWN ON THIS DWG FOR REF ONLY. 3) IMPEDANCE CONTROL REQUIRED. Microstrip 100-Ohm Dif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"
- board text added: "Front Side"
- board text added: "Hole Size"
- board text added: "L1 (Sig, PWR)"
- board text added: "L2 (GND)"
- board text added: "L3 (Sig, PWR)"
- board text added: "L4 (Sig, PWR)"
- board text added: "L5 (GND)"
- board text added: "L6 (Sig, PWR)"
- board text added: "PCB3D_BR_BOARDNAME"
- board text added: "PCB3D_TL_BOARDNAME"
- board text added: "Plated"
- board text added: "Plated Plated Plated Plated Plated Plated Plated Plated Plated Unplated"
- board text added: "Symbol"
- board text added: "THT SMD Total"
- board text added: "TP? TP? TP?"
- board text added: "Top Assembly (Scale 1:1)"
- board text added: "Top Fabrication (Scale 1:1)"
- board text added: "Top Test Points (Scale 1:1)"
- board text added: "Top View"
- board text added: "Total"
- board text removed: "?? ?? ?? ??"
- board text removed: "??mm"
- board text removed: "??mm (??oz)"
- board text removed: "FABRICATION NOTES (CONT.) 3) IMPEDANCE CONTROL REQUIRED. ? Microstrip ???-Ohm Differential (L? ref. L?, L? ref. L?) ??mm width, ??mm spacing 4) CONFIRM TRACE WIDTHS AND SPACINGS. 5) DESIGN GEOMETRY MINIMUM FEATURE SIZES: TRACE WIDTH ?? mm TRACE TO TRACE ?? mm MIN. HOLE (plated) ?? mm MIN. HOLE (unplated) ?? mm ANNULAR RING ?? mm COPPER TO HOLE ?? mm COPPER TO EDGE ?? mm HOLE TO HOLE ?? mm"
- board text removed: "FABRICATION NOTES (UNLESS OTHERWISE SPECIFIED) 1) 2)"
- board text removed: "L1 (??)"
- board text removed: "L2 (??)"
- board text removed: "L3 (??"
- board text removed: "L4 (??)"
- board text removed: "L5 (??)"
- board text removed: "L6 (??)"
- board text removed: "PCB3D_BR_Board_Name"
- board text removed: "PCB3D_TL_Board_Name"
- board text removed: "TP?? TP?? TP?? TP??"
